File: eagle/MotionSign.brd (EAGLE design)
At the start: 85.9 x 47.6 mm, 76 parts, among them Q1 16MHZ, U1 ATMEGA328, U2 L7805CDT-TR, U3 NCS36000, U4 PIR, U5 WS2801, U6 SPX3819, U7 NJVMJD2955T4G, U8 TXB0108PWR, U9 LCD-HD4478020X4-4HOLES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

Commit message: V0 of board
Parts:
- U9: device HD44780LCD:LCD-20X4-4HOLES -> HD44780LCD:LCD-20X4-1HOLE_NOSILK
- moved CTRST 1.02 mm to (117.1, 48.4)
- moved JP1 0.51 mm to (110.9, 49.1)
Routing:
- net VCC: track 288.9 -> 287.1 mm
- net VO: track 40.6 -> 39.6 mm
- net RXI: track 34.0 -> 33.2 mm
- net GND: vias 21 -> 22
Other:
- outline, holes or cut-outs redrawn
- board text added: "<-InTentss=Designs-> ||-MotionSign V0-||"
- board text added: "MotionSign V0"

Commit message: Slight board improvemnents
Parts:
- moved C14 7.41 mm to (70.1, 28.7), turned to 180 degrees
- moved C17 2.62 mm to (55.6, 40.3)
- moved C16 1.63 mm to (55.6, 35.9)
Routing:
- net VCC: track 287.1 -> 283.0 mm, vias 10 -> 8
- net 3.3V: track 71.5 -> 70.2 mm
