File: eagle/RemoteMotion/RemoteMotion.brd (EAGLE design)
At the start: 22.2 x 111.1 mm, 7 parts, among them J1 1

Commit message: Move to managed libarary for 3d parts
Parts:
- C1, C2: device rcl:C0805 -> RemoteMotion:C0805
- J1: device SparkFun-Connectors:JST-4-PTH -> RemoteMotion:JST-4-PTH
- LED1, LED2: device adafruit:WS2812B -> RemoteMotion:WS2812B
- R1: device rcl:R0805 -> RemoteMotion:R0805
- VR1: device SparkFun-Resistors:SLIDER-XLARGE -> RemoteMotion:SLIDER-XLARGE
Changed lines of the file:
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@@
 <?xml version="1.0" encoding="utf-8"?>
 <!DOCTYPE eagle SYSTEM "eagle.dtd">
-<eagle version="8.7.1">
+<eagle version="9.0.0">
 <drawing>
 <settings>
@@
 </layers>
 <board>
-<fusionsync huburn="a.cGVyc29uYWw6dWUyOGVmNjE0" projecturn="a.cGVyc29uYWw6dWUyOGVmNjE0IzIwMTgwMjIwMTE4NzI5NDc2" f3durn="urn:adsk.wipprod:dm.lineage:ZVttfNo7SJCkZL0V-kmSbQ" pcbguid="5a444160-fa68-4918-bfc4-b2eae5542b7b" lastpulledtime="" lastsyncedchangeguid="083b8e31-3dd0-4c27-0395-8cbbb61285e1"/>
+<fusionsync huburn="a.cGVyc29uYWw6dWUyOGVmNjE0" projecturn="a.cGVyc29uYWw6dWUyOGVmNjE0IzIwMTgwMjIwMTE4NzI5NDc2" f3durn="urn:adsk.wipprod:dm.lineage:ZVttfNo7SJCkZL0V-kmSbQ" pcbguid="5a444160-fa68-4918-bfc4-b2eae5542b7b" lastpulledtime="" lastsyncedchangeguid="61a6c252-1898-274f-7170-c01252bd9a9a"/>
 <plain>
 <wire x1="0" y1="107.95" x2="0" y2="3.175" width="0" layer="20"/>
@@
 </autorouter>
 <elements>
-<element name="J1" library="SparkFun-Connectors" package="JST-4-PTH" value="1" x="11.176" y="103.886" smashed="yes">
+<element name="J1" library="RemoteMotion" library_urn="urn:adsk.eagle:library:2810894" package="JST-4-PTH" package3d_urn="urn:adsk.eagle:package:2811204/1" value="1" x="11.176" y="103.886" smashed="yes">
 <attribute name="NAME" x="9.779" y="107.315" size="0.508" layer="25" font="vector" ratio="20"/>
 <attribute name="PROD_ID" value="WIRE-13531" x="11.176" y="103.886" size="1.778" layer="27" display="off"/>
 <attribute name="SF_ID" value="PRT-09916" x="11.176" y="103.886" size="1.778" layer="27" display="off"/>
 </element>
-<element name="LED1" library="adafruit" package="WS2812B" value="WS2812B5050" x="11.176" y="99.06" smashed="yes" rot="R180">
+<element name="LED1" library="RemoteMotion" library_urn="urn:adsk.eagle:library:2810894" package="WS2812B" package3d_urn="urn:adsk.eagle:package:2811216/1" value="WS2812B5050" x="11.176" y="99.06" smashed="yes" rot="R180">
 <attribute name="NAME" x="14.2875" y="98.2345" size="0.508" layer="25" ratio="10" rot="R90"/>
 </element>
-<element name="VR1" library="SparkFun-Resistors" package="SLIDER-XLARGE" value="10k" x="11.176" y="51.308" rot="R270">
+<element name="VR1" library="RemoteMotion" library_urn="urn:adsk.eagle:library:2810894" package="SLIDER-XLARGE" package3d_urn="urn:adsk.eagle:package:2811214/2" value="10k" x="11.176" y="51.308" rot="R270">
 <attribute name="PROD_ID" value="RES-09484" x="11.176" y="51.308" size="1.778" layer="27" rot="R270" display="off"/>
 <attribute name="SF_SKU" value="COM-09119" x="11.176" y="51.308" size="1.778" layer="27" rot="R270" display="off"/>
 </element>
-<element name="R1" library="rcl" library_urn="urn:adsk.eagle:library:334" package="R0805" package3d_urn="urn:adsk.eagle:package:23553/2" value="300" x="16.764" y="98.806" smashed="yes" rot="R270">
+<element name="R1" library="RemoteMotion" library_urn="urn:adsk.eagle:library:2810894" package="R0805" package3d_urn="urn:adsk.eagle:package:2811399/2" value="300" x="16.764" y="98.806" smashed="yes" rot="R270">
 <attribute name="NAME" x="16.51" y="96.52" size="0.508" layer="25"/>
 <attribute name="SPICEPREFIX" value="R" x="16.764" y="98.806" size="1.778" layer="27" rot="R270" display="off"/>
 <attribute name="VALUE" x="16.256" y="100.838" size="0.508" layer="27"/>
 </element>
-<element name="C1" library="rcl" library_urn="urn:adsk.eagle:library:334" package="C0805" package3d_urn="urn:adsk.eagle:package:23617/2" value="0.1uF" x="6.35" y="99.06" smashed="yes" rot="R270">
+<element name="C1" library="RemoteMotion" library_urn="urn:adsk.eagle:library:2810894" package="C0805" package3d_urn="urn:adsk.eagle:package:2811338/2" value="0.1uF" x="6.35" y="99.06" smashed="yes" rot="R270">
 <attribute name="NAME" x="6.096" y="101.092" size="0.508" layer="25"/>
 <attribute name="SPICEPREFIX" value="C" x="6.35" y="99.06" size="1.778" layer="27" rot="R270" display="off"/>
 <attribute name="VALUE" x="5.588" y="96.393" size="0.508" layer="27"/>
 </element>
-<element name="LED2" library="adafruit" package="WS2812B" value="WS2812B5050" x="10.16" y="3.556" smashed="yes">
+<element name="LED2" library="RemoteMotion" library_urn="urn:adsk.eagle:library:2810894" package="WS2812B" package3d_urn="urn:adsk.eagle:package:2811216/1" value="WS2812B5050" x="10.16" y="3.556" smashed="yes">
 <attribute name="NAME" x="7.4295" y="2.7305" size="0.508" layer="25" ratio="10" rot="R90"/>
 </element>
-<element name="C2" library="rcl" library_urn="urn:adsk.eagle:library:334" package="C0805" package3d_urn="urn:adsk.eagle:package:23617/2" value="0.1uF" x="14.986" y="3.556" smashed="yes" rot="R90">
+<element name="C2" library="RemoteMotion" library_urn="urn:adsk.eagle:library:2810894" package="C0805" package3d_urn="urn:adsk.eagle:package:2811338/2" value="0.1uF" x="14.986" y="3.556" smashed="yes" rot="R90">
 <attribute name="NAME" x="15.367" y="1.778" size="0.508" layer="25" rot="R180"/>
 <attribute name="SPICEPREFIX" value="C" x="14.986" y="3.556" size="1.778" layer="27" rot="R90" display="off"/>
